Commit message: Update URDF descriptions of robot cell, robot with EE and combined xacro file

File: robot_description_pkg/urdf/isaac_robot_cell_macro.xacro (robot description, xacro)
@@ -42,5 +42,5 @@
         name="charuco"
         parent="world"
-        xyz="0.5 0 0.794"
+        xyz="0.4 0 0.794"
         rpy="${pi} 0 ${-pi/2}"
         size="0.3"
@@ -51,5 +51,5 @@
       name="apriltag_0"
       parent="world"
-      xyz="0.75 -0.2 0.794"
+      xyz="0.65 -0.175 0.794"
       rpy="${pi} 0 ${-pi/2}"
       size="0.1"
@@ -59,5 +59,5 @@
       name="apriltag_1"
       parent="world"
-      xyz="0.75 0.2 0.794"
+      xyz="0.65 0.175 0.794"
       rpy="${pi} 0 ${-pi/2}"
       size="0.1"

File: robot_description_pkg/urdf/robot_cell.urdf.xacro (robot description, xacro)
@@ -1,4 +1,4 @@
 <?xml version="1.0"?>
-<robot name="my_robot_cell" xmlns:xacro="http://ros.org/wiki/xacro">
+<robot name="robot" xmlns:xacro="http://ros.org/wiki/xacro">
   <xacro:include filename="$(find robot_description_pkg)/urdf/robot_eef_macro.xacro"/>
   <xacro:include filename="$(find robot_description_pkg)/urdf/isaac_robot_cell_macro.xacro"/>
@@ -31,5 +31,5 @@
   >
     <xacro:if value="$(arg use_isaac)">
-      <origin xyz="0.15 -0.7 1.05" rpy="0 0 0" />
+      <origin xyz="0.3 -0.7 1.05" rpy="0 0 0" />
     </xacro:if>
     <xacro:unless value="$(arg use_isaac)">

File: robot_description_pkg/urdf/robot_eef_macro.xacro (robot description, xacro)
@@ -32,4 +32,8 @@
     <!-- End-Effector Attachment -->
     <link name="${tf_prefix}ee">
+      <inertial>
+        <mass value="1.0"/>
+        <inertia ixx="1e-9" iyy="1e-9" izz="1e-9" ixy="0" ixz="0" iyz="0"/>
+      </inertial>
       <visual>
         <geometry>
@@ -40,4 +44,9 @@
         </material>
       </visual>
+      <collision>
+        <geometry>
+          <mesh filename="package://robot_description_pkg/meshes/end_effector.stl" scale="0.001 0.001 0.001"/>
+        </geometry>
+      </collision>
     </link>
     <joint name="tool0_to_ee" type="fixed">
@@ -46,4 +55,16 @@
       <origin xyz="0 0 -0.0425" rpy="0 0 ${-pi/2}"/>
     </joint>
+    <!-- TCP Virtual Link -->
+    <link name="${tf_prefix}tcp">
+      <inertial>
+        <mass value="1e-6"/>
+        <inertia ixx="1e-9" iyy="1e-9" izz="1e-9" ixy="0" ixz="0" iyz="0"/>
+      </inertial>
+    </link>
+    <joint name="ee_to_tcp" type="fixed">
+      <parent link="${tf_prefix}ee"/>
+      <child link="${tf_prefix}tcp"/>
+      <origin xyz="0 0 0.28385" rpy="0 0 ${pi/2}"/>
+    </joint>
   </xacro:macro>
 </robot>
