Commit message: Add end-effector to robot model. Update RViz configs

File: robot_description_pkg/urdf/robot_eef_macro.xacro (robot description, xacro)
@@ -15,5 +15,5 @@
     safety_k_position:=20
     ">
-    <!--This will create the specific robot-->
+    <!--This will create the specific robot -->
     <xacro:ur_robot
       name="${ur_type}"
@@ -30,4 +30,20 @@
       <xacro:insert_block name="origin" />
     </xacro:ur_robot>
+    <!-- End-Effector Attachment -->
+    <link name="${tf_prefix}ee">
+      <visual>
+        <geometry>
+          <mesh filename="package://robot_description_pkg/meshes/end_effector.stl" scale="0.001 0.001 0.001"/>
+        </geometry>
+        <material name="grey">
+          <color rgba="0.7 0.7 0.7 1.0"/>
+        </material>
+      </visual>
+    </link>
+    <joint name="tool0_to_ee" type="fixed">
+      <parent link="${tf_prefix}tool0"/>
+      <child link="${tf_prefix}ee"/>
+      <origin xyz="0 0 -0.0425" rpy="0 0 ${-pi/2}"/>
+    </joint>
   </xacro:macro>
 </robot>

Commit message: Update robot EEF model and ground truth TCP transform from camera

File: robot_description_pkg/urdf/robot_eef_macro.xacro (robot description, xacro)
@@ -33,10 +33,10 @@
     <link name="${tf_prefix}ee">
       <inertial>
-        <mass value="1.0"/>
+        <mass value="1e-6"/>
         <inertia ixx="1e-9" iyy="1e-9" izz="1e-9" ixy="0" ixz="0" iyz="0"/>
       </inertial>
       <visual>
         <geometry>
-          <mesh filename="package://robot_description_pkg/meshes/end_effector.stl" scale="0.001 0.001 0.001"/>
+          <mesh filename="package://robot_description_pkg/meshes/end_effector.dae" scale="0.001 0.001 0.001"/>
         </geometry>
         <material name="grey">
@@ -46,5 +46,5 @@
       <collision>
         <geometry>
-          <mesh filename="package://robot_description_pkg/meshes/end_effector.stl" scale="0.001 0.001 0.001"/>
+          <mesh filename="package://robot_description_pkg/meshes/end_effector.dae" scale="0.001 0.001 0.001"/>
         </geometry>
       </collision>
@@ -65,5 +65,5 @@
       <parent link="${tf_prefix}ee"/>
       <child link="${tf_prefix}tcp"/>
-      <origin xyz="0 0 0.28385" rpy="0 0 ${pi/2}"/>
+      <origin xyz="0 0 0.2713" rpy="0 0 ${pi/2}"/>
     </joint>
   </xacro:macro>
